File: Schematic/Schematic.kicad_sch (KiCad schematic)
At the start: 168 parts, among them J1 Barrel_Jack, Q1 S8550, Q2 S8550, Q3 S8550, Q4 S8550, SW1 SW_Push, U1 GPS_Neo-6M, U2 DS1307, U3 L7805

Commit message: Schematic minor update
Parts:
- removed R12: 1k, symbol Device:R_Small_US
Connections:
- net DOT: now also D71.2 (A), D72.2 (A), D73.2 (A), D74.2 (A)
Changed lines of the file:
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@@
     (company "University of Kelaniya")
     (comment 1 "Department of Physics and Electronics")
-    (comment 2 "version: 1.0")
+    (comment 2 "version: 1.0.1")
     (comment 3 "Description: The clock automatically synchronizes its time once everyday with the GPS time")
     (comment 4 "Project Name: GPS CLOCK")
@@
     (stroke (width 0) (type default) (color 0 0 0 0))
   )
-  (wire (pts (xy 198.12 87.63) (xy 198.12 88.9))
+  (wire (pts (xy 198.12 92.71) (xy 198.12 95.25))
     (stroke (width 0) (type default) (color 0 0 0 0))
   )
@@
     (stroke (width 0) (type default) (color 0 0 0 0))
   )
-  (wire (pts (xy 198.12 93.98) (xy 198.12 95.25))
-    (stroke (width 0) (type default) (color 0 0 0 0))
-  )
   (wire (pts (xy 74.93 132.08) (xy 74.93 130.81))
     (stroke (width 0) (type default) (color 0 0 0 0))
@@
     )
   )
-  (global_label "DOT" (shape input) (at 198.12 87.63 90) (fields_autoplaced)
+  (global_label "DOT" (shape input) (at 198.12 92.71 90) (fields_autoplaced)
     (effects (font (size 1.27 1.27) italic) (justify left))
-    (property "Intersheet References" "${INTERSHEET_REFS}" (id 0) (at 198.0406 81.3932 90)
+    (property "Intersheet References" "${INTERSHEET_REFS}" (id 0) (at 198.0406 86.4732 90)
       (effects (font (size 1.27 1.27) italic) (justify left) hide)
     )
@@
       (effects (font (size 1.27 1.27)) hide)
     )
-    (property "Value" "+5V" (id 1) (at 67.31 69.85 0))
+    (property "Value" "+5V" (id 1) (at 66.04 69.85 0))
     (property "Footprint" "" (id 2) (at 67.31 73.66 0)
       (effects (font (size 1.27 1.27)) hide)
@@
       (effects (font (size 1.27 1.27)) hide)
     )
-    (property "Value" "+3.3V" (id 1) (at 72.39 69.85 0))
+    (property "Value" "+3.3V" (id 1) (at 71.12 69.85 0))
     (property "Footprint" "" (id 2) (at 69.85 73.66 0)
       (effects (font (size 1.27 1.27)) hide)
@@
     (pin "2")
   )
-  (symbol (lib_id "Device:R_Small_US") (at 198.12 91.44 180) (unit 1)
-    (in_bom yes) (on_board yes)
-    (property "Reference" "R12" (id 0) (at 200.66 90.17 0))
-    (property "Value" "1k" (id 1) (at 200.66 92.71 0))
-    (property "Footprint" "" (id 2) (at 198.12 91.44 0)
-      (effects (font (size 1.27 1.27)) hide)
-    )
-    (property "Datasheet" "~" (id 3) (at 198.12 91.44 0)
-      (effects (font (size 1.27 1.27)) hide)
-    )
-    (pin "1")
-    (pin "2")
-  )
   (symbol (lib_id "Device:LED_Small") (at 262.89 80.01 270) (mirror x) (unit 1)
     (in_bom yes) (on_board yes)
@@
       (reference "R11") (unit 1) (value "1k") (footprint "")
     )
-    (path "/bea67be3-8821-405c-bf18-8817260af9c2"
-      (reference "R12") (unit 1) (value "1k") (footprint "")
-    )
     (path "/ac9345ec-8f3a-4f80-ae34-7ed4b4fa2048"
